File: schematics/MrReflow/MrReflow.kicad_pcb (KiCad board)
At the start: 2 copper layers, 15 parts, among them U1 IRM-05-5, U2 WeMos_mini

Commit message: layout adjustments
Parts:
- moved H1 7.75 mm to (148.0, 40.6)
- moved H2 7.41 mm to (179.1, 40.6)
Routing:
- net (no net): track 0.00 -> 126.0 mm
- net Net-(H2-Pad1): track 12.5 -> 13.8 mm
Other:
- board outline added: 40 x 97.2 mm
- net class Default: trace_width 2 -> 0.2
Changed lines of the file:
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@@
-(kicad_pcb (version 20171130) (host pcbnew 5.0.1)
+(kicad_pcb (version 20171130) (host pcbnew "(5.0.0)")
   (general
     (thickness 1.6)
-    (drawings 0)
-    (tracks 72)
+    (drawings 1)
+    (tracks 81)
     (zones 0)
     (modules 15)
@@
   (page A4)
   (layers
-    (0 F.Cu signal)
+    (0 F.Cu signal hide)
     (31 B.Cu signal)
-    (32 B.Adhes user)
-    (33 F.Adhes user)
-    (34 B.Paste user)
-    (35 F.Paste user)
-    (36 B.SilkS user)
-    (37 F.SilkS user)
-    (38 B.Mask user)
-    (39 F.Mask user)
-    (40 Dwgs.User user)
-    (41 Cmts.User user)
-    (42 Eco1.User user)
-    (43 Eco2.User user)
+    (32 B.Adhes user hide)
+    (33 F.Adhes user hide)
+    (34 B.Paste user hide)
+    (35 F.Paste user hide)
+    (36 B.SilkS user hide)
+    (37 F.SilkS user hide)
+    (38 B.Mask user hide)
+    (39 F.Mask user hide)
+    (40 Dwgs.User user hide)
+    (41 Cmts.User user hide)
+    (42 Eco1.User user hide)
+    (43 Eco2.User user hide)
     (44 Edge.Cuts user)
-    (45 Margin user)
-    (46 B.CrtYd user)
-    (47 F.CrtYd user)
-    (48 B.Fab user)
-    (49 F.Fab user)
+    (45 Margin user hide)
+    (46 B.CrtYd user hide)
+    (47 F.CrtYd user hide)
+    (48 B.Fab user hide)
+    (49 F.Fab user hide)
   )
   (setup
-    (last_trace_width 2)
+    (last_trace_width 0.2)
     (trace_clearance 0.2)
     (zone_clearance 0.508)
@@
     (solder_mask_min_width 0.25)
     (aux_axis_origin 0 0)
-    (visible_elements FFFFFD67)
+    (visible_elements 7FFFFFFF)
     (pcbplotparams
-      (layerselection 0x010fc_ffffffff)
+      (layerselection 0x01008_ffffffff)
       (usegerberextensions false)
       (usegerberattributes false)
@@
       (outputformat 1)
       (mirror false)
-      (drillshape 1)
+      (drillshape 0)
       (scaleselection 1)
-      (outputdirectory ""))
+      (outputdirectory "cnc"))
   )
   (net 0 "")
@@
   (net_class Default "This is the default net class."
     (clearance 0.2)
-    (trace_width 2)
+    (trace_width 0.2)
     (via_dia 0.8)
     (via_drill 0.4)
@@
   )
   (module Connector_Pin:Pin_D1.0mm_L10.0mm (layer F.Cu)
-    (at 175.26 34.29)
+    (at 179.07 40.64)
     (descr "solder Pin_ diameter 1.0mm, hole diameter 1.0mm (press fit), length 10.0mm")
     (tags "solder Pin_ press fit")
@@
   )
   (module Connector_Pin:Pin_D1.0mm_L10.0mm (layer F.Cu)
-    (at 152.4 34.29)
+    (at 147.955 40.64)
     (descr "solder Pin_ diameter 1.0mm, hole diameter 1.0mm (press fit), length 10.0mm")
     (tags "solder Pin_ press fit")
@@
       (net 16 "Net-(U2-Pad9)"))
   )
+  (gr_poly (pts (xy 181.61 135.255) (xy 181.61 38.1) (xy 141.605 38.1) (xy 141.605 135.255)) (layer Edge.Cuts) (width 0.15))
+  (segment (start 144.145 46.99) (end 143.25001 46.99) (width 0.2) (layer F.Cu) (net 0))
+  (segment (start 160.02 46.99) (end 144.145 46.99) (width 0.2) (layer F.Cu) (net 0))
+  (segment (start 158.115 47.625) (end 183.13999 47.625) (width 0.2) (layer F.Cu) (net 0))
+  (segment (start 183.13999 47.625) (end 143.25001 47.625) (width 0.2) (layer F.Cu) (net 0))
+  (segment (start 143.25001 47.625) (end 143.51 47.625) (width 0.2) (layer F.Cu) (net 0))
+  (segment (start 160.655 46.355) (end 160.655 36.195) (width 0.2) (layer F.Cu) (net 0))
+  (segment (start 160.02 46.99) (end 160.655 46.99) (width 0.2) (layer F.Cu) (net 0))
+  (segment (start 160.655 36.195) (end 160.655 46.99) (width 0.2) (layer F.Cu) (net 0))
+  (segment (start 160.655 46.99) (end 183.13999 46.99) (width 0.2) (layer F.Cu) (net 0))
   (segment (start 154.94 120.65) (end 152.4 120.65) (width 2) (layer B.Cu) (net 3))
   (segment (start 153.67 91.7) (end 150.19999 95.17001) (width 2) (layer B.Cu) (net 3))
@@
   (segment (start 168.595505 104.14) (end 171.135505 104.14) (width 2) (layer B.Cu) (net 19))
   (segment (start 157.48 104.14) (end 160.02 104.14) (width 2) (layer B.Cu) (net 20))
-  (segment (start 154.58 36.47) (end 152.4 34.29) (width 2) (layer B.Cu) (net 21))
-  (segment (start 154.58 40.44) (end 154.58 36.47) (width 2) (layer B.Cu) (net 21))
-  (segment (start 169.11 40.44) (end 175.26 34.29) (width 2) (layer B.Cu) (net 22))
-  (segment (start 165.33 40.44) (end 169.11 40.44) (width 2) (layer B.Cu) (net 22))
+  (segment (start 148.155 40.44) (end 147.955 40.64) (width 2) (layer F.Cu) (net 21))
+  (segment (start 154.58 40.44) (end 148.155 40.44) (width 2) (layer B.Cu) (net 21))
+  (segment (start 178.87 40.44) (end 179.07 40.64) (width 2) (layer F.Cu) (net 22))
+  (segment (start 165.33 40.44) (end 178.87 40.44) (width 2) (layer B.Cu) (net 22))
 )
